Commit message: 优化B1 moveit控制

File: mercury_b1_moveit/config/gazebo_firefighter.urdf (robot description, URDF)
Before this commit: robot firefighter, 18 links, 17 joints
Links:
- link base: geometry collision cylinder length=0.14 radius=0.043; visual mesh filename=package://mercury_description/urdf/mercury_b1/base.dae
- link link1_L: geometry collision cylinder length=0.035 radius=0.023; visual mesh filename=package://mercury_description/urdf/mercury_b1/joint1_L.dae
- link link1_R: geometry collision cylinder length=0.035 radius=0.023; visual mesh filename=package://mercury_description/urdf/mercury_b1/joint1_R.dae
- link link2_L: geometry collision cylinder length=0.035 radius=0.023; visual mesh filename=package://mercury_description/urdf/mercury_b1/joint2_L.dae
- link link2_R: geometry collision cylinder length=0.035 radius=0.023; visual mesh filename=package://mercury_description/urdf/mercury_b1/joint2_R.dae
- link link3_L: geometry collision cylinder length=0.03 radius=0.023; visual mesh filename=package://mercury_description/urdf/mercury_b1/joint3_L.dae
- link link3_R: geometry collision cylinder length=0.03 radius=0.023; visual mesh filename=package://mercury_description/urdf/mercury_b1/joint3_R.dae
- link link4_L: geometry collision cylinder length=0.035 radius=0.023; visual mesh filename=package://mercury_description/urdf/mercury_b1/joint4_L.dae
- link link4_R: geometry collision cylinder length=0.035 radius=0.023; visual mesh filename=package://mercury_description/urdf/mercury_b1/joint4_R.dae
- link link5_L: geometry collision cylinder length=0.06 radius=0.023; visual mesh filename=package://mercury_description/urdf/mercury_b1/joint5_L.dae
- link link5_R: geometry collision cylinder length=0.06 radius=0.023; visual mesh filename=package://mercury_description/urdf/mercury_b1/joint5_R.dae
- link link6_L: geometry collision cylinder length=0.05 radius=0.023; visual mesh filename=package://mercury_description/urdf/mercury_b1/joint6_L.dae
- link link6_R: geometry collision cylinder length=0.05 radius=0.023; visual mesh filename=package://mercury_description/urdf/mercury_b1/joint6_R.dae
- link link7_L: geometry collision cylinder length=0.004 radius=0.023; visual mesh filename=package://mercury_description/urdf/mercury_b1/joint7_L.dae
- link link7_R: geometry collision cylinder length=0.004 radius=0.023; visual mesh filename=package://mercury_description/urdf/mercury_b1/joint7_R.dae
- link link_body: geometry collision cylinder length=0.14 radius=0.033; visual mesh filename=package://mercury_description/urdf/mercury_b1/body.dae
- link link_eye: geometry collision cylinder length=0.08 radius=0.003; visual mesh filename=package://mercury_description/urdf/mercury_b1/head_eye.dae
- link link_head: geometry collision cylinder length=0.05 radius=0.023; visual mesh filename=package://mercury_description/urdf/mercury_b1/head.dae
Joints:
- joint body: limit lower=-2.0594 upper=2.0594 effort=1000.0 velocity=0 -> lower=-2.059 upper=2.0594 effort=1000.0 velocity=0; origin xyz= 0 0 0.22    rpy=0 0 0 -> xyz= 0 0 0.231    rpy=0 0 0
- joint eye: limit lower=0 upper=0.8377 effort=1000.0 velocity=0 -> lower=-1.04 upper=0 effort=1000.0 velocity=0
- joint head: axis  0 0 1 ->  0 0 -1; limit lower=-2.4085 upper=3.2812 effort=1000.0 velocity=0 -> lower=-2.408 upper=3.2812 effort=1000.0 velocity=0
- joint joint1_L: limit lower=-3.1066 upper=3.1066 effort=1000.0 velocity=0 -> lower=-2.879 upper=2.879 effort=1000.0 velocity=0
- joint joint1_R: limit lower=-3.1066 upper=3.1066 effort=1000.0 velocity=0 -> lower=-2.879 upper=2.879 effort=1000.0 velocity=0
- joint joint2_L: limit lower=-1.4311 upper=2.2689 effort=1000.0 velocity=0 -> lower=-0.959 upper=1.658 effort=1000.0 velocity=0
- joint joint2_R: limit lower=-1.4311 upper=2.2689 effort=1000.0 velocity=0 -> lower=-0.959 upper=1.658 effort=1000.0 velocity=0
- joint joint3_L: limit lower=-3.1066 upper=3.1066 effort=1000.0 velocity=0 -> lower=-2.879 upper=2.879 effort=1000.0 velocity=0
- joint joint3_R: limit lower=-3.1066 upper=3.1066 effort=1000.0 velocity=0 -> lower=-2.879 upper=2.879 effort=1000.0 velocity=0
- joint joint4_L: limit lower=-3.0543 upper=0.2617 effort=1000.0 velocity=0 -> lower=-3.019 upper=0.087 effort=1000.0 velocity=0
- joint joint4_R: limit lower=-3.0543 upper=0.2617 effort=1000.0 velocity=0 -> lower=-3.019 upper=0.087 effort=1000.0 velocity=0
- joint joint5_L: limit lower=-3.1066 upper=3.1066 effort=1000.0 velocity=0 -> lower=-2.879 upper=2.879 effort=1000.0 velocity=0
- joint joint5_R: limit lower=-3.1066 upper=3.1066 effort=1000.0 velocity=0 -> lower=-2.879 upper=2.879 effort=1000.0 velocity=0
- joint joint6_L: limit lower=-0.0174 upper=2.9321 effort=1000.0 velocity=0 -> lower=-0.3490 upper=4.6251 effort=1000.0 velocity=0
- joint joint6_R: limit lower=-0.0174 upper=2.9321 effort=1000.0 velocity=0 -> lower=-0.3490 upper=4.6251 effort=1000.0 velocity=0
- joint joint7_L: limit lower=-3.1066 upper=3.1066 effort=1000.0 velocity=0 -> lower=-3.14 upper=3.14 effort=1000.0 velocity=0
- joint joint7_R: limit lower=-3.1066 upper=3.1066 effort=1000.0 velocity=0 -> lower=-3.14 upper=3.14 effort=1000.0 velocity=0

File: mercury_description/urdf/mercury_b1/mercury_b1_moveit.urdf (robot description, URDF)
Before this commit: robot firefighter, 18 links, 17 joints
Links:
- link base: geometry collision cylinder length=0.14 radius=0.043; visual mesh filename=package://mercury_description/urdf/mercury_b1/base.dae
- link link1_L: geometry collision cylinder length=0.035 radius=0.023; visual mesh filename=package://mercury_description/urdf/mercury_b1/joint1_L.dae
- link link1_R: geometry collision cylinder length=0.035 radius=0.023; visual mesh filename=package://mercury_description/urdf/mercury_b1/joint1_R.dae
- link link2_L: geometry collision cylinder length=0.035 radius=0.023; visual mesh filename=package://mercury_description/urdf/mercury_b1/joint2_L.dae
- link link2_R: geometry collision cylinder length=0.035 radius=0.023; visual mesh filename=package://mercury_description/urdf/mercury_b1/joint2_R.dae
- link link3_L: geometry collision cylinder length=0.03 radius=0.023; visual mesh filename=package://mercury_description/urdf/mercury_b1/joint3_L.dae
- link link3_R: geometry collision cylinder length=0.03 radius=0.023; visual mesh filename=package://mercury_description/urdf/mercury_b1/joint3_R.dae
- link link4_L: geometry collision cylinder length=0.035 radius=0.023; visual mesh filename=package://mercury_description/urdf/mercury_b1/joint4_L.dae
- link link4_R: geometry collision cylinder length=0.035 radius=0.023; visual mesh filename=package://mercury_description/urdf/mercury_b1/joint4_R.dae
- link link5_L: geometry collision cylinder length=0.06 radius=0.023; visual mesh filename=package://mercury_description/urdf/mercury_b1/joint5_L.dae
- link link5_R: geometry collision cylinder length=0.06 radius=0.023; visual mesh filename=package://mercury_description/urdf/mercury_b1/joint5_R.dae
- link link6_L: geometry collision cylinder length=0.05 radius=0.023; visual mesh filename=package://mercury_description/urdf/mercury_b1/joint6_L.dae
- link link6_R: geometry collision cylinder length=0.05 radius=0.023; visual mesh filename=package://mercury_description/urdf/mercury_b1/joint6_R.dae
- link link7_L: geometry collision cylinder length=0.004 radius=0.023; visual mesh filename=package://mercury_description/urdf/mercury_b1/joint7_L.dae
- link link7_R: geometry collision cylinder length=0.004 radius=0.023; visual mesh filename=package://mercury_description/urdf/mercury_b1/joint7_R.dae
- link link_body: geometry collision cylinder length=0.14 radius=0.033; visual mesh filename=package://mercury_description/urdf/mercury_b1/body.dae
- link link_eye: geometry collision cylinder length=0.08 radius=0.003; visual mesh filename=package://mercury_description/urdf/mercury_b1/head_eye.dae
- link link_head: geometry collision cylinder length=0.05 radius=0.023; visual mesh filename=package://mercury_description/urdf/mercury_b1/head.dae
