Commit message: B3 urdf adds joint quality parameters

File: mercury_description/urdf/mercury_b3/mercury_b3.urdf (robot description, URDF)
Before this commit: robot firefighter, 18 links, 17 joints
Links:
- added link world
- link base: mass None -> 3.2
- link link1_L: mass None -> 1.143
- link link1_R: mass None -> 1.143
- link link2_L: mass None -> 1.732
- link link2_R: mass None -> 1.732
- link link3_L: mass None -> 1.436
- link link3_R: mass None -> 1.436
- link link4_L: mass None -> 1.431
- link link4_R: mass None -> 1.431
- link link5_L: mass None -> 0.718
- link link5_R: mass None -> 0.718
- link link6_L: mass None -> 0.799
- link link6_R: mass None -> 0.799
- link link7_L: mass None -> 0.046
- link link7_R: mass None -> 0.046
- link link_body: mass None -> 3.018
- link link_eye: mass None -> 0.021
- link link_head: mass None -> 1.2
Joints:
- added joint world_to_base: type fixed, parent world, child base, origin xyz=0 0 0 rpy=0 0 0
