Commit message: update joint limit

File: mercury_description/urdf/mercury_a1/mercury_a1.urdf (robot description, URDF)
Before this commit: robot firefighter, 8 links, 7 joints
Joints:
- joint joint1_to_base: limit lower=-3.1066 upper=3.1066 effort=1000.0 velocity=0 -> lower=-2.879 upper=2.879 effort=1000.0 velocity=0
- joint joint2_to_joint1: limit lower=-1.4311 upper=2.2689 effort=1000.0 velocity=0 -> lower=-0.959 upper=1.658 effort=1000.0 velocity=0
- joint joint3_to_joint2: limit lower=-3.1066 upper=3.1066 effort=1000.0 velocity=0 -> lower=-2.879 upper=2.879 effort=1000.0 velocity=0
- joint joint4_to_joint3: limit lower=-3.0543 upper=0.2617 effort=1000.0 velocity=0 -> lower=-3.019 upper=0.087 effort=1000.0 velocity=0
- joint joint5_to_joint4: limit lower=-3.1066 upper=3.1066 effort=1000.0 velocity=0 -> lower=-2.879 upper=2.879 effort=1000.0 velocity=0
- joint joint7_to_joint6: limit lower=-3.1066 upper=3.1066 effort=1000.0 velocity=0 -> lower=-3.14 upper=3.14 effort=1000.0 velocity=0

File: mercury_description/urdf/mercury_b1/mercury_b1.urdf (robot description, URDF)
Before this commit: robot firefighter, 18 links, 17 joints
Joints:
- joint body: limit lower=-2.0594 upper=2.0594 effort=1000.0 velocity=0 -> lower=-2.059 upper=2.0594 effort=1000.0 velocity=0
- joint eye: limit lower=0 upper=0.83 effort=1000.0 velocity=0 -> lower=-1.04 upper=0 effort=1000.0 velocity=0
- joint head: limit lower=-2.4085 upper=3.2812 effort=1000.0 velocity=0 -> lower=-2.321 upper=3.2812 effort=1000.0 velocity=0
- joint joint1_L: limit lower=-3.1066 upper=3.1066 effort=1000.0 velocity=0 -> lower=-2.879 upper=2.879 effort=1000.0 velocity=0
- joint joint1_R: limit lower=-3.1066 upper=3.1066 effort=1000.0 velocity=0 -> lower=-2.879 upper=2.879 effort=1000.0 velocity=0
- joint joint2_L: limit lower=-1.4311 upper=2.2689 effort=1000.0 velocity=0 -> lower=-0.959 upper=1.658 effort=1000.0 velocity=0
- joint joint2_R: limit lower=-1.4311 upper=2.2689 effort=1000.0 velocity=0 -> lower=-0.959 upper=1.658 effort=1000.0 velocity=0
- joint joint3_L: limit lower=-3.1066 upper=3.1066 effort=1000.0 velocity=0 -> lower=-2.879 upper=2.879 effort=1000.0 velocity=0
- joint joint3_R: limit lower=-3.1066 upper=3.1066 effort=1000.0 velocity=0 -> lower=-2.879 upper=2.879 effort=1000.0 velocity=0
- joint joint4_L: limit lower=-3.0543 upper=0.2617 effort=1000.0 velocity=0 -> lower=-3.019 upper=0.087 effort=1000.0 velocity=0
- joint joint4_R: limit lower=-3.0543 upper=0.2617 effort=1000.0 velocity=0 -> lower=-3.019 upper=0.087 effort=1000.0 velocity=0
- joint joint5_L: limit lower=-3.1066 upper=3.1066 effort=1000.0 velocity=0 -> lower=-2.879 upper=2.879 effort=1000.0 velocity=0
- joint joint5_R: limit lower=-3.1066 upper=3.1066 effort=1000.0 velocity=0 -> lower=-2.879 upper=2.879 effort=1000.0 velocity=0
- joint joint7_L: limit lower=-3.1066 upper=3.1066 effort=1000.0 velocity=0 -> lower=-3.14 upper=3.14 effort=1000.0 velocity=0
- joint joint7_R: limit lower=-3.1066 upper=3.1066 effort=1000.0 velocity=0 -> lower=-3.14 upper=3.14 effort=1000.0 velocity=0

Commit message: 优化A1 moveit模型显示碰撞问题

File: mercury_description/urdf/mercury_a1/mercury_a1.urdf (robot description, URDF)
Before this commit: robot firefighter, 8 links, 7 joints
Links:
- link base: geometry collision cylinder length=0.07 radius=0.043; visual mesh filename=package://mercury_description/urdf/mercury_a1/base.dae
- link joint1: geometry collision cylinder length=0.02 radius=0.023; visual mesh filename=package://mercury_description/urdf/mercury_a1/joint1.dae
- link joint2: geometry collision cylinder length=0.035 radius=0.023; visual mesh filename=package://mercury_description/urdf/mercury_a1/joint2.dae
- link joint3: geometry collision cylinder length=0.02 radius=0.023; visual mesh filename=package://mercury_description/urdf/mercury_a1/joint3.dae
- link joint4: geometry collision cylinder length=0.035 radius=0.023; visual mesh filename=package://mercury_description/urdf/mercury_a1/joint4.dae
- link joint5: geometry collision cylinder length=0.06 radius=0.023; visual mesh filename=package://mercury_description/urdf/mercury_a1/joint5.dae
- link joint6: geometry collision cylinder length=0.05 radius=0.023; visual mesh filename=package://mercury_description/urdf/mercury_a1/joint6.dae
- link joint7: geometry collision cylinder length=0.004 radius=0.023; visual mesh filename=package://mercury_description/urdf/mercury_a1/joint7.dae

Commit message: perf(A1-ros):Mercury A1 updated URDF model file

File: mercury_description/urdf/mercury_a1/mercury_a1.urdf (robot description, URDF)
Before this commit: robot firefighter, 8 links, 7 joints
Links:
- link base: geometry collision cylinder length=0.07 radius=0.043; visual mesh filename=package://mercury_description/urdf/mercury_a1/BASE-W.dae
- link joint1: geometry collision cylinder length=0.01 radius=0.012; visual mesh filename=package://mercury_description/urdf/mercury_a1/J1-W.dae
- link joint2: geometry collision cylinder length=0.035 radius=0.023; visual mesh filename=package://mercury_description/urdf/mercury_a1/J2-W.dae
- link joint3: geometry collision cylinder length=0.02 radius=0.023; visual mesh filename=package://mercury_description/urdf/mercury_a1/J3-W.dae
- link joint4: geometry collision cylinder length=0.035 radius=0.023; visual mesh filename=package://mercury_description/urdf/mercury_a1/J4-W.STL
- link joint5: geometry collision cylinder length=0.06 radius=0.023; visual mesh filename=package://mercury_description/urdf/mercury_a1/J5-W.STL
Joints:
- joint joint1_to_base: origin xyz=0 0 0.175 rpy=0 0 0 -> xyz=0 0 0.17835 rpy=0 0 0
- joint joint2_to_joint1: limit lower=-0.959 upper=1.658 effort=1000.0 velocity=0 -> lower=-0.8726 upper=2.0943 effort=1000.0 velocity=0; origin xyz=0 0  0 rpy=-1.5708 0 0 -> xyz=0 -0.005 -0.01 rpy=-1.5708 0 0
- joint joint3_to_joint2: origin xyz=0 -0.11 0    rpy=1.5708 0 0 -> xyz=0 -0.134 0.004    rpy=1.5708 0 0
- joint joint4_to_joint3: limit lower=-3.019 upper=0.087 effort=1000.0 velocity=0 -> lower=-2.879 upper=0.087 effort=1000.0 velocity=0; origin xyz=0.03 0 0.095 rpy=-1.5708 0 3.14159 -> xyz=0.03 0 0.07 rpy=-1.5708 0 3.14159
- joint joint5_to_joint4: origin xyz=0.03 -0.126 0 rpy=1.5708 3.14159 0 -> xyz=0.031 -0.11 0 rpy=1.5708 3.14159 0
- joint joint6_to_joint5: limit lower=-0.0349 upper=2.9321 effort=1000.0 velocity=0 -> lower=-0.3490 upper=4.6251 effort=1000.0 velocity=0; origin xyz=0 0.0 0.08 rpy=1.5708 0 0 -> xyz=0 0.03 0.095 rpy=1.5708 0 0
- joint joint7_to_joint6: origin xyz=0.038 -0.046 0 rpy=1.5708 0 0 -> xyz=0.038 -0.045 0.025 rpy=1.5708 0 0

File: mercury_description/urdf/mercury_a1/mercury_a1_old.urdf (robot description, URDF)
Before this commit: robot firefighter, 9 links, 8 joints
Links:
- removed link three_gripper
- link base: geometry collision cylinder length=0.07 radius=0.043; visual mesh filename=package://mercury_description/urdf/mercury_a1/base.dae
- link joint1: geometry collision cylinder length=0.02 radius=0.023; visual mesh filename=package://mercury_description/urdf/mercury_a1/joint1.dae
- link joint2: geometry collision cylinder length=0.035 radius=0.023; visual mesh filename=package://mercury_description/urdf/mercury_a1/joint2.dae
- link joint3: geometry collision cylinder length=0.02 radius=0.023; visual mesh filename=package://mercury_description/urdf/mercury_a1/joint3.dae
- link joint4: geometry collision cylinder length=0.035 radius=0.023; visual mesh filename=package://mercury_description/urdf/mercury_a1/joint4.dae
- link joint5: geometry collision cylinder length=0.06 radius=0.023; visual mesh filename=package://mercury_description/urdf/mercury_a1/joint5.dae
Joints:
- removed joint gripper_to_joint7
- joint joint1_to_base: origin xyz=0 0 0.17835 rpy=0 0 0 -> xyz=0 0 0.175 rpy=0 0 0
- joint joint2_to_joint1: limit lower=-0.8726 upper=2.0943 effort=1000.0 velocity=0 -> lower=-0.959 upper=1.658 effort=1000.0 velocity=0; origin xyz=0 -0.005 -0.01 rpy=-1.5708 0 0 -> xyz=0 0  0 rpy=-1.5708 0 0
- joint joint3_to_joint2: origin xyz=0 -0.134 0.004    rpy=1.5708 0 0 -> xyz=0 -0.11 0    rpy=1.5708 0 0
- joint joint4_to_joint3: limit lower=-2.879 upper=0.087 effort=1000.0 velocity=0 -> lower=-3.019 upper=0.087 effort=1000.0 velocity=0; origin xyz=0.03 0 0.07 rpy=-1.5708 0 3.14159 -> xyz=0.03 0 0.095 rpy=-1.5708 0 3.14159
- joint joint5_to_joint4: origin xyz=0.031 -0.11 0 rpy=1.5708 3.14159 0 -> xyz=0.03 -0.126 0 rpy=1.5708 3.14159 0
- joint joint6_to_joint5: limit lower=-0.3490 upper=4.6251 effort=1000.0 velocity=0 -> lower=-0.0349 upper=2.9321 effort=1000.0 velocity=0; origin xyz=0 0.03 0.095 rpy=1.5708 -1.5708 0 -> xyz=0 0.0 0.08 rpy=1.5708 0 0
- joint joint7_to_joint6: origin xyz=0.038 -0.045 0.025 rpy=1.5708 0 0 -> xyz=0.038 -0.046 0 rpy=1.5708 0 0

Commit message: fix(A1-ROS):updated URDF model file

File: mercury_description/urdf/mercury_a1/mercury_a1.urdf (robot description, URDF)
Before this commit: robot firefighter, 8 links, 7 joints
Links:
- link joint6: geometry collision cylinder length=0.05 radius=0.023; visual mesh filename=package://mercury_description/urdf/mercury_a1/J6-W.dae
- link joint7: geometry collision cylinder length=0.004 radius=0.023; visual mesh filename=package://mercury_description/urdf/mercury_a1/J7-W.dae
Joints:
- joint joint7_to_joint6: origin xyz=0.038 -0.045 0.025 rpy=1.5708 0 0 -> xyz=0.042 -0.043 0.029 rpy=1.5708 0 0

File: mercury_description/urdf/mercury_a1/mercury_a1_three_gripper.urdf (robot description, URDF)
Before this commit: robot firefighter, 9 links, 8 joints
Links:
- link joint6: geometry collision cylinder length=0.05 radius=0.023; visual mesh filename=package://mercury_description/urdf/mercury_a1/J6-W.dae
- link joint7: geometry collision cylinder length=0.004 radius=0.023; visual mesh filename=package://mercury_description/urdf/mercury_a1/J7-W.dae
Joints:
- joint joint7_to_joint6: origin xyz=0.038 -0.045 0.025 rpy=1.5708 0 0 -> xyz=0.042 -0.043 0.029 rpy=1.5708 0 0
