Commit message: feat(A1-URDF): update A1 URDF file

File: mercury_description/urdf/mercury_a1/mercury_a1.urdf (robot description, URDF)
Before this commit: robot firefighter, 8 links, 7 joints
Links:
- removed link base
- removed link joint1
- removed link joint2
- removed link joint3
- removed link joint4
- removed link joint5
- removed link joint6
- removed link joint7
- added link Link2, mass 0.36178; collision mesh filename=package://mercury_description/urdf/mercury_a1/meshes/Link2.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; visual mesh filename=package://mercury_description/urdf/mercury_a1/meshes/Link2.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
- added link Link3, mass 0.28631; collision mesh filename=package://mercury_description/urdf/mercury_a1/meshes/Link3.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; visual mesh filename=package://mercury_description/urdf/mercury_a1/meshes/Link3.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
- added link Link4, mass 0.242339225037204; collision mesh filename=package://mercury_description/urdf/mercury_a1/meshes/Link4.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; visual mesh filename=package://mercury_description/urdf/mercury_a1/meshes/Link4.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
- added link Link5, mass 0.155939982030202; collision mesh filename=package://mercury_description/urdf/mercury_a1/meshes/Link5.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; visual mesh filename=package://mercury_description/urdf/mercury_a1/meshes/Link5.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
- added link Link6, mass 0.227233689100569; collision mesh filename=package://mercury_description/urdf/mercury_a1/meshes/Link6.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; visual mesh filename=package://mercury_description/urdf/mercury_a1/meshes/Link6.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
- added link Link7, mass 0.0300324439188857; collision mesh filename=package://mercury_description/urdf/mercury_a1/meshes/Link7.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; visual mesh filename=package://mercury_description/urdf/mercury_a1/meshes/Link7.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
- added link base_link, mass 0.480011489444113; collision mesh filename=package://mercury_description/urdf/mercury_a1/meshes/base_l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; visual mesh filename=package://mercury_description/urdf/mercury_a1/meshes/base_l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
- added link link1, mass 0.33317; collision mesh filename=package://mercury_description/urdf/mercury_a1/meshes/link1.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; visual mesh filename=package://mercury_description/urdf/mercury_a1/meshes/link1.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
Joints:
- removed joint joint1_to_base
- removed joint joint2_to_joint1
- removed joint joint3_to_joint2
- removed joint joint4_to_joint3
- removed joint joint5_to_joint4
- removed joint joint6_to_joint5
- removed joint joint7_to_joint6
- added joint joint1: type revolute, parent base_link, child link1, origin xyz=0 0 0.08364 rpy=0 0 0, axis 0 0 1, limit lower=-2.8798 upper=2.8798 effort=0 velocity=0
- added joint joint2: type revolute, parent link1, child Link2, origin xyz=0 0 0 rpy=-1.5708 0 0, axis 0 0 1, limit lower=-0.8727 upper=2.0944 effort=0 velocity=0
- added joint joint3: type revolute, parent Link2, child Link3, origin xyz=0 -0.20199 0 rpy=1.5708 0 0, axis 0 0 1, limit lower=-2.8798 upper=2.8798 effort=0 velocity=0
- added joint joint4: type revolute, parent Link3, child Link4, origin xyz=0.02953 0 0 rpy=1.5708 0 0, axis 0 0 1, limit lower=-2.8798 upper=0.0873 effort=0 velocity=0
- added joint joint5: type revolute, parent Link4, child Link5, origin xyz=-0.02953 0.20602 0 rpy=-1.5708 0 0, axis 0 0 1, limit lower=-2.8798 upper=2.8798 effort=0 velocity=0
- added joint joint6: type revolute, parent Link5, child Link6, origin xyz=0 0 0 rpy=1.5708 0 0, axis 0 0 1, limit lower=-0.3491 upper=4.6251 effort=0 velocity=0
- added joint joint7: type revolute, parent Link6, child Link7, origin xyz=0.042 -0.05101 0 rpy=1.5708 0 0, axis 0 0 1, limit lower=-3.1416 upper=3.1416 effort=0 velocity=0

File: mercury_description/urdf/mercury_a1/mercury_a1_three_gripper.urdf (robot description, URDF)
Before this commit: robot firefighter, 9 links, 8 joints
Links:
- removed link base
- removed link joint1
- removed link joint2
- removed link joint3
- removed link joint4
- removed link joint5
- removed link joint6
- removed link joint7
- removed link three_gripper
- added link Link2, mass 0.36178; collision mesh filename=package://mercury_description/urdf/mercury_a1/meshes/Link2.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; visual mesh filename=package://mercury_description/urdf/mercury_a1/meshes/Link2.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
- added link Link3, mass 0.28631; collision mesh filename=package://mercury_description/urdf/mercury_a1/meshes/Link3.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; visual mesh filename=package://mercury_description/urdf/mercury_a1/meshes/Link3.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
- added link Link4, mass 0.242339225037204; collision mesh filename=package://mercury_description/urdf/mercury_a1/meshes/Link4.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; visual mesh filename=package://mercury_description/urdf/mercury_a1/meshes/Link4.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
- added link Link5, mass 0.155939982030202; collision mesh filename=package://mercury_description/urdf/mercury_a1/meshes/Link5.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; visual mesh filename=package://mercury_description/urdf/mercury_a1/meshes/Link5.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
- added link Link6, mass 0.227233689100569; collision mesh filename=package://mercury_description/urdf/mercury_a1/meshes/Link6.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; visual mesh filename=package://mercury_description/urdf/mercury_a1/meshes/Link6.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
- added link Link7, mass 0.0300324439188857; collision mesh filename=package://mercury_description/urdf/mercury_a1/meshes/Link7.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; visual mesh filename=package://mercury_description/urdf/mercury_a1/meshes/Link7.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
- added link Link_gripper; collision cylinder length=0.004 radius=0.023; visual mesh filename=package://mercury_description/urdf/three_gripper/three_myha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
- added link base_link, mass 0.480011489444113; collision mesh filename=package://mercury_description/urdf/mercury_a1/meshes/base_l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; visual mesh filename=package://mercury_description/urdf/mercury_a1/meshes/base_l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
- added link link1, mass 0.33317; collision mesh filename=package://mercury_description/urdf/mercury_a1/meshes/link1.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; visual mesh filename=package://mercury_description/urdf/mercury_a1/meshes/link1.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
Joints:
- removed joint joint1_to_base
- removed joint joint2_to_joint1
- removed joint joint3_to_joint2
- removed joint joint4_to_joint3
- removed joint joint5_to_joint4
- removed joint joint6_to_joint5
- removed joint joint7_to_joint6
- added joint joint1: type revolute, parent base_link, child link1, origin xyz=0 0 0.08364 rpy=0 0 0, axis 0 0 1, limit lower=-2.8798 upper=2.8798 effort=0 velocity=0
- added joint joint2: type revolute, parent link1, child Link2, origin xyz=0 0 0 rpy=-1.5708 0 0, axis 0 0 1, limit lower=-0.8727 upper=2.0944 effort=0 velocity=0
- added joint joint3: type revolute, parent Link2, child Link3, origin xyz=0 -0.20199 0 rpy=1.5708 0 0, axis 0 0 1, limit lower=-2.8798 upper=2.8798 effort=0 velocity=0
- added joint joint4: type revolute, parent Link3, child Link4, origin xyz=0.02953 0 0 rpy=1.5708 0 0, axis 0 0 1, limit lower=-2.8798 upper=0.0873 effort=0 velocity=0
- added joint joint5: type revolute, parent Link4, child Link5, origin xyz=-0.02953 0.20602 0 rpy=-1.5708 0 0, axis 0 0 1, limit lower=-2.8798 upper=2.8798 effort=0 velocity=0
- added joint joint6: type revolute, parent Link5, child Link6, origin xyz=0 0 0 rpy=1.5708 0 0, axis 0 0 1, limit lower=-0.3491 upper=4.6251 effort=0 velocity=0
- added joint joint7: type revolute, parent Link6, child Link7, origin xyz=0.042 -0.05101 0 rpy=1.5708 0 0, axis 0 0 1, limit lower=-3.1416 upper=3.1416 effort=0 velocity=0
- joint gripper_to_joint7: child three_gripper -> Link_gripper; origin xyz=0.0 0.0 0.05 rpy=0 0 0 -> xyz=0.0 0.0 0.0 rpy=0 0 0; parent joint7 -> Link7
