Commit message: Update mercury_b1.urdf

File: mercury_description/urdf/mercury_b1/mercury_b1.urdf (robot description, URDF)
Before this commit: robot firefighter, 18 links, 17 joints
Joints:
- joint head: limit lower=-2.321 upper=3.2812 effort=1000.0 velocity=0 -> lower=-2.408 upper=3.2812 effort=1000.0 velocity=0
- joint joint6_L: limit lower=-0.0349 upper=2.9321 effort=1000.0 velocity=0 -> lower=-0.3490 upper=4.6251 effort=1000.0 velocity=0
- joint joint6_R: limit lower=-0.0349 upper=2.9321 effort=1000.0 velocity=0 -> lower=-0.3490 upper=4.6251 effort=1000.0 velocity=0

Commit message: 更新水星B1 URDF关节限位

File: mercury_description/urdf/mercury_b1/mercury_b1.urdf (robot description, URDF)
Before this commit: robot firefighter, 18 links, 17 joints
Joints:
- joint joint2_L: limit lower=-0.959 upper=1.658 effort=1000.0 velocity=0 -> lower=-0.8726 upper=2.0943 effort=1000.0 velocity=0
- joint joint2_R: limit lower=-0.959 upper=1.658 effort=1000.0 velocity=0 -> lower=-0.8726 upper=2.0943 effort=1000.0 velocity=0
- joint joint4_L: limit lower=-3.019 upper=0.087 effort=1000.0 velocity=0 -> lower=-2.879 upper=0.087 effort=1000.0 velocity=0
- joint joint4_R: limit lower=-3.019 upper=0.087 effort=1000.0 velocity=0 -> lower=-2.879 upper=0.087 effort=1000.0 velocity=0

File: mercury_description/urdf/mercury_b1/mercury_b1_moveit.urdf (robot description, URDF)
Before this commit: robot firefighter, 18 links, 17 joints
Joints:
- joint joint2_L: limit lower=-0.959 upper=1.658 effort=1000.0 velocity=0 -> lower=-0.8726 upper=2.0943 effort=1000.0 velocity=0
- joint joint2_R: limit lower=-0.959 upper=1.658 effort=1000.0 velocity=0 -> lower=-0.8726 upper=2.0943 effort=1000.0 velocity=0
- joint joint4_L: limit lower=-3.019 upper=0.087 effort=1000.0 velocity=0 -> lower=-2.879 upper=0.087 effort=1000.0 velocity=0
- joint joint4_R: limit lower=-3.019 upper=0.087 effort=1000.0 velocity=0 -> lower=-2.879 upper=0.087 effort=1000.0 velocity=0

File: mercury_description/urdf/mercury_b1/mercury_b1_pro_gripper.urdf (robot description, URDF)
Before this commit: robot firefighter, 32 links, 31 joints
Joints:
- joint joint2_L: limit lower=-0.959 upper=1.658 effort=1000.0 velocity=0 -> lower=-0.8726 upper=2.0943 effort=1000.0 velocity=0
- joint joint2_R: limit lower=-0.959 upper=1.658 effort=1000.0 velocity=0 -> lower=-0.8726 upper=2.0943 effort=1000.0 velocity=0
- joint joint4_L: limit lower=-3.019 upper=0.087 effort=1000.0 velocity=0 -> lower=-2.879 upper=0.087 effort=1000.0 velocity=0
- joint joint4_R: limit lower=-3.019 upper=0.087 effort=1000.0 velocity=0 -> lower=-2.879 upper=0.087 effort=1000.0 velocity=0

File: mercury_description/urdf/mercury_b1/mercury_b1_pro_gripper_new.urdf (robot description, URDF)
Before this commit: robot firefighter, 32 links, 31 joints
Joints:
- joint joint2_L: limit lower=-0.959 upper=1.658 effort=1000.0 velocity=0 -> lower=-0.8726 upper=2.0943 effort=1000.0 velocity=0
- joint joint2_R: limit lower=-0.959 upper=1.658 effort=1000.0 velocity=0 -> lower=-0.8726 upper=2.0943 effort=1000.0 velocity=0
- joint joint4_L: limit lower=-3.019 upper=0.087 effort=1000.0 velocity=0 -> lower=-2.879 upper=0.087 effort=1000.0 velocity=0
- joint joint4_R: limit lower=-3.019 upper=0.087 effort=1000.0 velocity=0 -> lower=-2.879 upper=0.087 effort=1000.0 velocity=0

Commit message: perf(B1-URDF): Updated B1 to URDF Version 2.0

File: mercury_description/urdf/mercury_b1/mercury_b1.urdf (robot description, URDF)
Before this commit: robot firefighter, 18 links, 17 joints
Links:
- removed link base
- removed link link1_L
- removed link link1_R
- removed link link2_L
- removed link link2_R
- removed link link3_L
- removed link link3_R
- removed link link4_L
- removed link link4_R
- removed link link5_L
- removed link link5_R
- removed link link6_L
- removed link link6_R
- removed link link7_L
- removed link link7_R
- removed link link_body
- removed link link_eye
- removed link link_head
- added link L1_Link, mass 0.333175155332311; collision mesh filename=package://mercury_description/urdf/mercury_b1/meshes/L1_Lin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; visual mesh filename=package://mercury_description/urdf/mercury_b1/meshes/L1_Lin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
- added link L2_Link, mass 0.361775197812871; collision mesh filename=package://mercury_description/urdf/mercury_b1/meshes/L2_Lin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; visual mesh filename=package://mercury_description/urdf/mercury_b1/meshes/L2_Lin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
- added link L3_Link, mass 0.28631136916664; collision mesh filename=package://mercury_description/urdf/mercury_b1/meshes/L3_Lin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; visual mesh filename=package://mercury_description/urdf/mercury_b1/meshes/L3_Lin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
- added link L4_Link, mass 0.242339322350328; collision mesh filename=package://mercury_description/urdf/mercury_b1/meshes/L4_Lin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; visual mesh filename=package://mercury_description/urdf/mercury_b1/meshes/L4_Lin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
- added link L5_Link, mass 0.155941224668293; collision mesh filename=package://mercury_description/urdf/mercury_b1/meshes/L5_Lin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; visual mesh filename=package://mercury_description/urdf/mercury_b1/meshes/L5_Lin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
- added link L6_Link, mass 0.227232628149454; collision mesh filename=package://mercury_description/urdf/mercury_b1/meshes/L6_Lin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; visual mesh filename=package://mercury_description/urdf/mercury_b1/meshes/L6_Lin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
- added link L7_Link, mass 0.0300324441314696; collision mesh filename=package://mercury_description/urdf/mercury_b1/meshes/L7_Lin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; visual mesh filename=package://mercury_description/urdf/mercury_b1/meshes/L7_Lin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
- added link R1_Link, mass 0.333174849091845; collision mesh filename=package://mercury_description/urdf/mercury_b1/meshes/R1_Lin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; visual mesh filename=package://mercury_description/urdf/mercury_b1/meshes/R1_Lin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
- added link R2_Link, mass 0.36177164559734; collision mesh filename=package://mercury_description/urdf/mercury_b1/meshes/R2_Lin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; visual mesh filename=package://mercury_description/urdf/mercury_b1/meshes/R2_Lin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
- added link R3_Link, mass 0.286312926844065; collision mesh filename=package://mercury_description/urdf/mercury_b1/meshes/R3_Lin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; visual mesh filename=package://mercury_description/urdf/mercury_b1/meshes/R3_Lin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
- added link R4_Link, mass 0.242325622607969; collision mesh filename=package://mercury_description/urdf/mercury_b1/meshes/R4_Lin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; visual mesh filename=package://mercury_description/urdf/mercury_b1/meshes/R4_Lin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
- added link R5_Link, mass 0.155938691268561; collision mesh filename=package://mercury_description/urdf/mercury_b1/meshes/R5_Lin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; visual mesh filename=package://mercury_description/urdf/mercury_b1/meshes/R5_Lin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
- added link R6_Link, mass 0.227233635909737; collision mesh filename=package://mercury_description/urdf/mercury_b1/meshes/R6_Lin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; visual mesh filename=package://mercury_description/urdf/mercury_b1/meshes/R6_Lin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
- added link R7_Link, mass 0.0300324441325877; collision mesh filename=package://mercury_description/urdf/mercury_b1/meshes/R7_Lin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; visual mesh filename=package://mercury_description/urdf/mercury_b1/meshes/R7_Lin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
- added link base_link, mass 2.88524669227858; collision mesh filename=package://mercury_description/urdf/mercury_b1/meshes/base_L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; visual mesh filename=package://mercury_description/urdf/mercury_b1/meshes/base_L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
- added link body_Link, mass 1.84312182388031; collision mesh filename=package://mercury_description/urdf/mercury_b1/meshes/body_L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; visual mesh filename=package://mercury_description/urdf/mercury_b1/meshes/body_L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
- added link camera_Link, mass 0.0215402832809272; collision mesh filename=package://mercury_description/urdf/mercury_b1/meshes/camera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; visual mesh filename=package://mercury_description/urdf/mercury_b1/meshes/camera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
- added link dummy_link
- added link head_Link, mass 1.19614017700233; collision mesh filename=package://mercury_description/urdf/mercury_b1/meshes/head_L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; visual mesh filename=package://mercury_description/urdf/mercury_b1/meshes/head_L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
Joints:
- removed joint eye
- removed joint joint1_L
- removed joint joint1_R
- removed joint joint2_L
- removed joint joint2_R
- removed joint joint3_L
- removed joint joint3_R
- removed joint joint4_L
- removed joint joint4_R
- removed joint joint5_L
- removed joint joint5_R
- removed joint joint6_L
- removed joint joint6_R
- removed joint joint7_L
- removed joint joint7_R
- added joint L1_joint: type revolute, parent body_Link, child L1_Link, origin xyz=-0.118497394816875 0.0182738890202244 0.188499999999995 rpy=1.57079632679493 -1.3613568165556 1.36135681655573, axis 0 0 -1, limit lower=-2.87 upper=2.87 effort=10000 velocity=2.61
- added joint L2_joint: type revolute, parent L1_Link, child L2_Link, origin xyz=0.0070916 0.0015074 -0.08215 rpy=1.5708 1.5271 1.7802, axis 0 0 -1, limit lower=-0.87 upper=2.09 effort=10000 velocity=2.61
- added joint L3_joint: type revolute, parent L2_Link, child L3_Link, origin xyz=0.119535751998164 -0.00522678221895016 -0.00824999999999831 rpy=-1.57079632679491 -0.161317342007266 -1.61449416830792, axis 0 0 1, limit lower=-2.87 upper=2.87 effort=10000 velocity=2.61
- added joint L4_joint: type revolute, parent L3_Link, child L4_Link, origin xyz=0.0302814729663858 -0.00241762176226584 0.0818500000000202 rpy=-1.5707963267949 -0.619422014804291 -2.98027531158253, axis 0 0 1, limit lower=-2.87 upper=0.0174 effort=10000 velocity=2.61
- added joint L5_joint: type revolute, parent L4_Link, child L5_Link, origin xyz=0.0701567904374146 -0.0475789413030669 -0.00825000000000015 rpy=-1.5707963267949 -0.69071648231178 0.619422013996731, axis 0 0 -1, limit lower=-2.87 upper=2.87 effort=10000 velocity=2.61
- added joint L6_joint: type revolute, parent L5_Link, child L6_Link, origin xyz=0.0183609223561629 -0.0222141605790311 -0.12603 rpy=-1.5707963267949 -1.26273791559162 0.69071648231178, axis 0 0 -1, limit lower=-2.87 upper=2.87 effort=10000 velocity=2.61
- added joint L7_joint: type revolute, parent L6_Link, child L7_Link, origin xyz=-0.0506977777847214 -0.0208039254363527 0.0283216918889004 rpy=1.5707963267949 0.253768150357354 -0.308058411203275, axis 0 0 1, limit lower=-2.87 upper=2.87 effort=10000 velocity=2.61
- added joint R1_joint: type revolute, parent body_Link, child R1_Link, origin xyz=0.118497394817623 0.0182738890154283 0.188499999999997 rpy=1.57079632679489 0.209439510239314 1.78023583699358, axis 0 0 1, limit lower=-2.87 upper=2.87 effort=10000 velocity=2.61
- added joint R2_joint: type revolute, parent R1_Link, child R2_Link, origin xyz=0.00161131160777349 -0.00758062716891239 0.0821499697613877 rpy=1.57079632679489 -1.37076011220364 0.209439510240489, axis 0 0 -1, limit lower=-0.87 upper=2.09 effort=10000 velocity=2.61
- added joint R3_joint: type revolute, parent R2_Link, child R3_Link, origin xyz=0.117264075564476 0.0237750256749663 -0.0082500000000002 rpy=1.5707963267949 0 1.77083254134537, axis 0 0 1, limit lower=-2.87 upper=2.87 effort=10000 velocity=2.61
- added joint R4_joint: type revolute, parent R3_Link, child R4_Link, origin xyz=-0.0294999999999995 0.00775000000000126 0.0818500000000005 rpy=1.57079632679492 1.37133227810459 -3.14159265358977, axis 0 0 1, limit lower=-2.87 upper=0.0174 effort=10000 velocity=2.61
- added joint R5_joint: type revolute, parent R4_Link, child R5_Link, origin xyz=-0.0920710602715785 -0.011484370268659 -0.00824999999999898 rpy=-1.5707963267949 -0.175965359389049 -1.77026037548521, axis 0 0 -1, limit lower=-2.87 upper=2.87 effort=10000 velocity=2.61
- added joint R6_joint: type revolute, parent R5_Link, child R6_Link, origin xyz=-0.00452001489370575 0.0254212876416742 -0.118453681718218 rpy=1.5707963267949 -1.19343079707769 -2.96562729420074, axis 0 0 -1, limit lower=-2.87 upper=2.87 effort=10000 velocity=2.61
- added joint R7_joint: type revolute, parent R6_Link, child R7_Link, origin xyz=-0.0318714873450072 -0.0445788770640032 -0.0253216918888982 rpy=1.5707963267949 1.48578825159432 0.252653002267418, axis 0 0 1, limit lower=-2.87 upper=2.87 effort=10000 velocity=2.61
- added joint camera: type revolute, parent head_Link, child camera_Link, origin xyz=-0.0388569238285446 -0.0372589398101035 -0.0260001449065854 rpy=-1.57079632679487 0.130499600987671 3.14159265358979, axis 0 0 1, limit lower=-0.95 upper=0 effort=10000 velocity=1.13
- added joint dummy: type fixed, parent dummy_link, child base_link
- joint body: axis  0 0 1 -> 0 0 1; child link_body -> body_Link; limit lower=-2.059 upper=2.0594 effort=1000.0 velocity=0 -> lower=-2.79 upper=2.79 effort=10000 velocity=1.13; origin xyz= 0 0 0.231    rpy=0 0 0 -> xyz=-0.0411232379784645 -0.0411232379784645 0.1567 rpy=0 0 3.14159265358979; parent base -> base_link
- joint head: axis  0 0 -1 -> 0 0 1; child link_head -> head_Link; limit lower=-2.408 upper=3.2812 effort=1000.0 velocity=0 -> lower=-1.22 upper=3.83 effort=10000 velocity=1.13; origin xyz= 0 0 0.22    rpy=0 0 0 -> xyz=0 0 0.234300000000004 rpy=-3.14159265358979 0 -1.5707963267949; parent link_body -> body_Link
